File: hardware/usb-port/usb-port.kicad_pcb (KiCad board)
At the start: 2 copper layers, 26 x 7.6 mm, 11 parts, among them J1 USB4105-GF-A, M1 M2 clearance, M2 M2 clearance

Commit message: hardware: add USB-C port schematic and verify PCB parity
Parts:
- H1, H2, H3, H4, H5, H6: footprint (none) -> RaceRemote_USB:WirePad_D0.8mm
- J1: footprint USB_C_Receptacle_GCT_USB4105-xx-A_16P_TopMnt_Horizontal -> RaceRemote_USB:USB_C_Receptacle_GCT_USB4105-xx-A_16P_TopMnt_Horizontal
- M1, M2: footprint (none) -> RaceRemote_USB:MountingHole_2.4mm
- R1, R2: footprint R_0603_1608Metric -> RaceRemote_USB:R_0603_1608Metric
Connections:
- J1 pad A8: (no net) -> unconnected-(J1-SBU1-PadA8)
- J1 pad B8: (no net) -> unconnected-(J1-SBU2-PadB8)
Changed lines of the file:
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@@
 		)
 	)
-	(footprint ""
+	(footprint "RaceRemote_USB:WirePad_D0.8mm"
 		(layer "F.Cu")
 		(at 88.4 97)
@@
 		(embedded_fonts no)
 	)
-	(footprint "USB_C_Receptacle_GCT_USB4105-xx-A_16P_TopMnt_Horizontal"
+	(footprint "RaceRemote_USB:USB_C_Receptacle_GCT_USB4105-xx-A_16P_TopMnt_Horizontal"
 		(layer "F.Cu")
 		(at 100 100)
@@
 			)
 		)
-		(property "Datasheet" ""
+		(property "Datasheet" "https://gct.co/files/drawings/usb4105.pdf"
 			(at 0 0 0)
 			(unlocked yes)
@@
 			(layers "F.Cu" "F.Mask" "F.Paste")
 			(roundrect_rratio 0.25)
+			(net "unconnected-(J1-SBU1-PadA8)")
 		)
 		(pad "A9" smd roundrect
@@
 			(layers "F.Cu" "F.Mask" "F.Paste")
 			(roundrect_rratio 0.25)
+			(net "unconnected-(J1-SBU2-PadB8)")
 		)
 		(pad "B9" smd roundrect
@@
 		)
 	)
-	(footprint ""
+	(footprint "RaceRemote_USB:MountingHole_2.4mm"
 		(layer "F.Cu")
 		(at 92 99.825)
@@
 			)
 		)
+		(attr exclude_from_bom)
 		(duplicate_pad_numbers_are_jumpers no)
 		(pad "" np_thru_hole circle
@@
 		(embedded_fonts no)
 	)
-	(footprint ""
+	(footprint "RaceRemote_USB:WirePad_D0.8mm"
 		(layer "F.Cu")
 		(at 88.4 101.4)
@@
 		(embedded_fonts no)
 	)
-	(footprint ""
+	(footprint "RaceRemote_USB:WirePad_D0.8mm"
 		(layer "F.Cu")
 		(at 111.6 99.2)
@@
 		(embedded_fonts no)
 	)
-	(footprint ""
+	(footprint "RaceRemote_USB:MountingHole_2.4mm"
 		(layer "F.Cu")
 		(at 108 99.825)
@@
 			)
 		)
+		(attr exclude_from_bom)
 		(duplicate_pad_numbers_are_jumpers no)
 		(pad "" np_thru_hole circle
@@
 		(embedded_fonts no)
 	)
-	(footprint ""
+	(footprint "RaceRemote_USB:WirePad_D0.8mm"
 		(layer "F.Cu")
 		(at 111.6 97)
@@
 		(embedded_fonts no)
 	)
-	(footprint ""
+	(footprint "RaceRemote_USB:WirePad_D0.8mm"
 		(layer "F.Cu")
 		(at 111.6 101.4)
@@
 		(embedded_fonts no)
 	)
-	(footprint ""
+	(footprint "RaceRemote_USB:WirePad_D0.8mm"
 		(layer "F.Cu")
 		(at 88.4 99.2)
@@
 		(embedded_fonts no)
 	)
-	(footprint "R_0603_1608Metric"
+	(footprint "RaceRemote_USB:R_0603_1608Metric"
 		(layer "B.Cu")
 		(at 98.5 100.4 180)
@@
 		)
 	)
-	(footprint "R_0603_1608Metric"
+	(footprint "RaceRemote_USB:R_0603_1608Metric"
 		(layer "B.Cu")
 		(at 101.5 100.4 180)
