File: hardware/charge-core/charge-core.kicad_sch (KiCad schematic)
At the start: 21 parts, among them J101 QUALIFIED INPUT, J102 PROTECTED CHARGE PATH, J103 EXTERNAL CHARGE GATE, J104 EXTERNAL NTC 103AT-2, U101 BQ25886RGER

Commit message: hardware: isolate charger detection from external USB data lines
Parts:
- added R108: 0, symbol RaceRemote_Charge:R
- J101: value QUALIFIED INPUT -> QUALIFIED POWER ONLY; symbol RaceRemote_Charge:Conn_01x04 -> RaceRemote_Charge:Conn_01x02
Connections:
- net DM renamed CORE_DM
- net CORE_DM: now also R108.2; no longer J101.4 (Pin_4)
- net DP renamed CORE_DP
- net CORE_DP: now also R108.1; no longer J101.3 (Pin_3)
Other:
- note added: "CE_N pulled high: default charge OFF. OTG tied low. VSET floating: nominal 8.4V. 250mA is a proposed bench setting; LW charge limits and cell pinout remain unverified. No traction load on SYS_INTERNAL. Do not connect raw LW battery to this unfinished assembly. R108 configures local DCP detection. J101 is POWER ONLY; source permission comes from the external gate."
- note removed: "CE_N pulled high: default charge OFF. OTG tied low. VSET floating: nominal 8.4V. 250mA is a proposed bench setting; LW charge limits and cell pinout remain unverified. No traction load on SYS_INTERNAL. Do not connect raw LW battery to this unfinished assembly."
Changed lines of the file:
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@@
 (kicad_sch (version 20250901) (generator "raceremote")
  (paper "A3")
-(title_block (title "RaceRemote - BQ25886 charger core PROPOSAL") (date "2026-09-14") (rev "0.1") (company "vea.raceremote"))
+(title_block (title "RaceRemote - BQ25886 charger core PROPOSAL") (date "2026-09-14") (rev "0.2") (company "vea.raceremote"))
 (symbol (lib_id "RaceRemote_Charge:BQ25886RGE") (at 101.6 83.82 0) (unit 1) (in_bom yes) (on_board yes) (dnp no) (property "Reference" "U101" (at 101.6 58.42 0) (effects (font (size 1.27 1.27))))(property "Value" "BQ25886RGER" (at 101.6 55.88 0) (effects (font (size 1.27 1.27))))(property "Footprint" "Package_DFN_QFN:Texas_RGE0024H_VQFN-24-1EP_4x4mm_P0.5mm_EP2.7x2.7mm" (at 101.6 83.82 0) (hide yes) (effects (font (size 1.27 1.27))))(property "Datasheet" "https://www.ti.com/lit/gpn/bq25886" (at 101.6 83.82 0) (hide yes) (effects (font (size 1.27 1.27))))(pin "1")(pin "2")(pin "3")(pin "4")(pin "5")(pin "6")(pin "7")(pin "8")(pin "9")(pin "10")(pin "11")(pin "12")(pin "13")(pin "14")(pin "15")(pin "16")(pin "17")(pin "18")(pin "19")(pin "20")(pin "21")(pin "22")(pin "23")(pin "24")(pin "25")(instances (project "charge-core" (path "/c3551efd-fb3f-5092-85f3-8a45b4f3354f" (reference "U101") (unit 1)))))
 (wire (pts (xy 91.44 66.04) (xy 78.74 66.04)) (stroke (width 0) (type default)))
 (global_label "CHG_VBUS" (shape passive) (at 78.74 66.04 180) (effects (font (size 1.0 1.0)) (justify right)))
 (wire (pts (xy 91.44 71.12) (xy 78.74 71.12)) (stroke (width 0) (type default)))
-(global_label "DP" (shape passive) (at 78.74 71.12 180) (effects (font (size 1.0 1.0)) (justify right)))
+(global_label "CORE_DP" (shape passive) (at 78.74 71.12 180) (effects (font (size 1.0 1.0)) (justify right)))
 (wire (pts (xy 91.44 73.66) (xy 78.74 73.66)) (stroke (width 0) (type default)))
-(global_label "DM" (shape passive) (at 78.74 73.66 180) (effects (font (size 1.0 1.0)) (justify right)))
+(global_label "CORE_DM" (shape passive) (at 78.74 73.66 180) (effects (font (size 1.0 1.0)) (justify right)))
 (wire (pts (xy 91.44 88.9) (xy 78.74 88.9)) (stroke (width 0) (type default)))
 (global_label "CHG_GND" (shape passive) (at 78.74 88.9 180) (effects (font (size 1.0 1.0)) (justify right)))
@@
 (wire (pts (xy 330.2 224.79) (xy 330.2 232.41)) (stroke (width 0) (type default)))
 (global_label "CHG_GND" (shape passive) (at 330.2 232.41 0) (effects (font (size 1.0 1.0)) (justify left)))
-(symbol (lib_id "RaceRemote_Charge:Conn_01x04") (at 177.8 226.06 0) (unit 1) (in_bom yes) (on_board yes) (dnp no) (property "Reference" "J101" (at 177.8 220.98 0) (effects (font (size 1.27 1.27))))(property "Value" "QUALIFIED INPUT" (at 177.8 218.44 0) (effects (font (size 1.27 1.27))))(property "Footprint" "" (at 177.8 226.06 0) (hide yes) (effects (font (size 1.27 1.27))))(property "Datasheet" "" (at 177.8 226.06 0) (hide yes) (effects (font (size 1.27 1.27))))(pin "1")(pin "2")(pin "3")(pin "4")(instances (project "charge-core" (path "/c3551efd-fb3f-5092-85f3-8a45b4f3354f" (reference "J101") (unit 1)))))
-(wire (pts (xy 172.72 223.52) (xy 165.1 223.52)) (stroke (width 0) (type default)))
-(global_label "CHG_VBUS" (shape passive) (at 165.1 223.52 180) (effects (font (size 1.0 1.0)) (justify right)))
+(symbol (lib_id "RaceRemote_Charge:R") (at 50.8 114.3 0) (unit 1) (in_bom yes) (on_board yes) (dnp no) (property "Reference" "R108" (at 50.8 109.22 0) (effects (font (size 1.27 1.27))))(property "Value" "0" (at 60.96 114.3 0) (effects (font (size 1.27 1.27))))(property "Footprint" "" (at 50.8 114.3 0) (hide yes) (effects (font (size 1.27 1.27))))(property "Datasheet" "" (at 50.8 114.3 0) (hide yes) (effects (font (size 1.27 1.27))))(pin "1")(pin "2")(instances (project "charge-core" (path "/c3551efd-fb3f-5092-85f3-8a45b4f3354f" (reference "R108") (unit 1)))))
+(wire (pts (xy 50.8 110.49) (xy 50.8 102.87)) (stroke (width 0) (type default)))
+(global_label "CORE_DP" (shape passive) (at 50.8 102.87 0) (effects (font (size 1.0 1.0)) (justify left)))
+(wire (pts (xy 50.8 118.11) (xy 50.8 125.73)) (stroke (width 0) (type default)))
+(global_label "CORE_DM" (shape passive) (at 50.8 125.73 0) (effects (font (size 1.0 1.0)) (justify left)))
+(symbol (lib_id "RaceRemote_Charge:Conn_01x02") (at 177.8 226.06 0) (unit 1) (in_bom yes) (on_board yes) (dnp no) (property "Reference" "J101" (at 177.8 220.98 0) (effects (font (size 1.27 1.27))))(property "Value" "QUALIFIED POWER ONLY" (at 177.8 218.44 0) (effects (font (size 1.27 1.27))))(property "Footprint" "" (at 177.8 226.06 0) (hide yes) (effects (font (size 1.27 1.27))))(property "Datasheet" "" (at 177.8 226.06 0) (hide yes) (effects (font (size 1.27 1.27))))(pin "1")(pin "2")(instances (project "charge-core" (path "/c3551efd-fb3f-5092-85f3-8a45b4f3354f" (reference "J101") (unit 1)))))
 (wire (pts (xy 172.72 226.06) (xy 165.1 226.06)) (stroke (width 0) (type default)))
-(global_label "CHG_GND" (shape passive) (at 165.1 226.06 180) (effects (font (size 1.0 1.0)) (justify right)))
+(global_label "CHG_VBUS" (shape passive) (at 165.1 226.06 180) (effects (font (size 1.0 1.0)) (justify right)))
 (wire (pts (xy 172.72 228.6) (xy 165.1 228.6)) (stroke (width 0) (type default)))
-(global_label "DP" (shape passive) (at 165.1 228.6 180) (effects (font (size 1.0 1.0)) (justify right)))
-(wire (pts (xy 172.72 231.14) (xy 165.1 231.14)) (stroke (width 0) (type default)))
-(global_label "DM" (shape passive) (at 165.1 231.14 180) (effects (font (size 1.0 1.0)) (justify right)))
+(global_label "CHG_GND" (shape passive) (at 165.1 228.6 180) (effects (font (size 1.0 1.0)) (justify right)))
 (symbol (lib_id "RaceRemote_Charge:Conn_01x02") (at 254 220.98 0) (unit 1) (in_bom yes) (on_board yes) (dnp no) (property "Reference" "J102" (at 254 215.9 0) (effects (font (size 1.27 1.27))))(property "Value" "PROTECTED CHARGE PATH" (at 254 213.36 0) (effects (font (size 1.27 1.27))))(property "Footprint" "" (at 254 220.98 0) (hide yes) (effects (font (size 1.27 1.27))))(property "Datasheet" "" (at 254 220.98 0) (hide yes) (effects (font (size 1.27 1.27))))(pin "1")(pin "2")(instances (project "charge-core" (path "/c3551efd-fb3f-5092-85f3-8a45b4f3354f" (reference "J102") (unit 1)))))
 (wire (pts (xy 248.92 220.98) (xy 241.3 220.98)) (stroke (width 0) (type default)))
@@
 (global_label "SW" (shape passive) (at 152.4 264.16 0) (effects (font (size 1.0 1.0)) (justify left)))
 (text "Converter core only - source qualification, cell monitor/balancer and protection are separate." (at 25.4 20.32 0) (effects (font (size 2 2)) (justify left top)))
-(text "CE_N pulled high: default charge OFF. OTG tied low. VSET floating: nominal 8.4V.\n250mA is a proposed bench setting; LW charge limits and cell pinout remain unverified.\nNo traction load on SYS_INTERNAL. Do not connect raw LW battery to this unfinished assembly." (at 25.4 30.48 0) (effects (font (size 1.27 1.27)) (justify left top)))
+(text "CE_N pulled high: default charge OFF. OTG tied low. VSET floating: nominal 8.4V.\n250mA is a proposed bench setting; LW charge limits and cell pinout remain unverified.\nNo traction load on SYS_INTERNAL. Do not connect raw LW battery to this unfinished assembly.\nR108 configures local DCP detection. J101 is POWER ONLY; source permission comes from the external gate." (at 25.4 30.48 0) (effects (font (size 1.27 1.27)) (justify left top)))
 (text "C104/C105: >=44uF effective total at operating voltage. Nominal values are placeholders for MPN selection.\nGround: short analog returns and power-pad star per TI; high-current loops require PCB review.\nFlags describe power connectivity for ERC; they do not implement source checks or reverse protection." (at 25.4 279.4 0) (effects (font (size 1.0 1.0)) (justify left top)))
 (sheet_instances (path "/" (page "1"))) (embedded_fonts no))
