File: hardware/charge-permit/charge-permit.kicad_sch (KiCad schematic)
At the start: 13 parts, among them J401 FROM AUX, J402 FAULT SOURCES, J403 MCU INTERFACE, J404 TO FUTURE GATE, U401 SN74LVC1G74DCTR, U402 SN74LVC2G17DCKR, U403 TPS3808G33DBVR

Commit message: hardware: add conditional charger CD inhibit candidate
Parts:
- added C404, C405: 100n / 16V, symbol RaceRemote_Permit:C
- added R404: 47k / 1%, symbol RaceRemote_Permit:R
- added R405: 1M / 1%, symbol RaceRemote_Permit:R
- added U404, U405: TMUX1219DBVR, symbol RaceRemote_Permit:TMUX1219DBV
- J401: value FROM AUX -> AUX AND CHARGER BIAS; symbol RaceRemote_Permit:Conn_01x02 -> RaceRemote_Permit:Conn_01x04
- J404: value TO FUTURE GATE -> TO BQ25887 CD
Connections:
- net AUX_3V3: no longer C403.1, U403.3 (~{MR}), U403.6 (VDD)
- net FAULT_BUS_N: now also R405.1, U405.1 (SEL)
- net PERMIT_Q: now also U404.1 (SEL); no longer J404.1 (Pin_1)
- net USB_GND: now also J401.4 (Pin_4), C404.2, C405.2, R405.2, U404.3 (GND), U404.6 (S2 (SEL=1)), U405.3 (GND)
- new net CD_REQUEST: U404.5 (D), U405.6 (S2 (SEL=1))
- new net CHARGER_CD: J404.1 (Pin_1), R404.2, U405.5 (D)
- new net CHG_BIAS: C403.1, C404.1, C405.1, J401.3 (Pin_3), R404.1, U403.3 (~{MR}), U403.6 (VDD), U404.2 (VDD), U404.4 (S1 (SEL=0)), U405.2 (VDD), U405.4 (S1 (SEL=0))
Other:
- note added: "CHARGE-PERMIT-01 v0.2 - latch + CD signal actuator; complete charger NOT qualified"
- note added: "CHG_BIAS proposal: qualified charger-input rail 4.5..5.5V. Existing TPS25200 may clamp at 5.55V: NOT yet compatible. AUX 3.0..3.6V; SENSE falling nominal 3.07V. Delays/fast ramps/bias loss and restart still require measurement. No MCU, watchdog, INA300 or charger power stage here. This sheet does not authorize battery connection."
- note added: "FAULT LOW: U405 selects CHG_BIAS directly, even when Q is unknown. FAULT HIGH: U405 passes U404 output. CD LOW requires Q HIGH. Supervisor and both muxes use CHG_BIAS; U401/U402 use AUX. J401 changed to 4 pins. J404 is now active-HIGH CD, NOT PERMIT_Q."
- note removed: "AUX 3.0..3.6V proposal; supervisor falling nominal 3.07V. Below IC valid rails, outputs are NOT guaranteed. No MCU/watchdog/INA300/charger actuator here. PCB, timing, transient and deep-brownout qualification are open."
- note removed: "CHARGE-PERMIT-01 v0.1 - logical latch candidate, NOT a complete charger shutdown"
- title: RaceRemote - hardware permit latch PROPOSAL -> RaceRemote - permit latch and CD actuator PROPOSAL

Commit message: hardware: regulate charger inhibit bias independently from AUX
Parts:
- added C406: 1u / 50V, symbol RaceRemote_Permit:C
- added C407: 4.7u / 16V X7R, symbol RaceRemote_Permit:C
- added R406: 3.3k / 1%, symbol RaceRemote_Permit:R
- added U406: TPS70933DBVR, symbol RaceRemote_Permit:TPS70933DBV
- J401: value AUX AND CHARGER BIAS -> AUX AND CHARGER INPUT
Connections:
- net USB_GND: now also C406.2, C407.2, R406.2, U406.2 (GND)
- net CHG_BIAS renamed CHG_BIAS_3V3
- net CHG_BIAS_3V3: now also C407.1, R406.1, U406.5 (OUT); no longer J401.3 (Pin_3)
- new net CHG_SUPPLY_INPUT: C406.1, J401.3 (Pin_3), U406.1 (IN)
- no-connect marks 2 -> 4
Other:
- note added: "CHARGE-PERMIT-01 v0.3 - latch + regulated CD bias; complete charger NOT qualified"
- note added: "CHG_BIAS_3V3 is now regulated 3.3V, target 3.0..3.6V. U406 tolerates the conditional 5.55V input clamp. AUX 3.0..3.6V; SENSE falling nominal 3.07V. Delays/fast ramps/bias loss and restart still require measurement. No MCU, watchdog, INA300 or charger power stage here. This sheet does not authorize battery connection."
- note added: "FAULT LOW: U405 selects CHG_BIAS_3V3 directly, even when Q is unknown. FAULT HIGH: U405 passes U404 output. CD LOW requires Q HIGH. Supervisor and both muxes use CHG_BIAS_3V3; U401/U402 use AUX. J401.3 is now U406 input. J404 is active-HIGH CD, NOT PERMIT_Q."
- note removed: "CHARGE-PERMIT-01 v0.2 - latch + CD signal actuator; complete charger NOT qualified"
- note removed: "CHG_BIAS proposal: qualified charger-input rail 4.5..5.5V. Existing TPS25200 may clamp at 5.55V: NOT yet compatible. AUX 3.0..3.6V; SENSE falling nominal 3.07V. Delays/fast ramps/bias loss and restart still require measurement. No MCU, watchdog, INA300 or charger power stage here. This sheet does not authorize battery connection."
- note removed: "FAULT LOW: U405 selects CHG_BIAS directly, even when Q is unknown. FAULT HIGH: U405 passes U404 output. CD LOW requires Q HIGH. Supervisor and both muxes use CHG_BIAS; U401/U402 use AUX. J401 changed to 4 pins. J404 is now active-HIGH CD, NOT PERMIT_Q."

Commit message: hardware: add charger MCU interface and default-low request stages
Parts:
- R402: value 10k / 1% -> 47k / 1%
Other:
- note added: "CHARGE-PERMIT-01 v0.4 - ARM pull-down 47k for MCU inverter; complete charger NOT qualified"
- note removed: "CHARGE-PERMIT-01 v0.3 - latch + regulated CD bias; complete charger NOT qualified"
Changed lines of the file:
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@@
 (kicad_sch (version 20250901) (generator "raceremote")
  (paper "A2")
-(title_block (title "RaceRemote - permit latch and CD actuator PROPOSAL") (date "2026-09-14") (rev "0.3") (company "vea.raceremote"))
+(title_block (title "RaceRemote - permit latch and CD actuator PROPOSAL") (date "2026-09-14") (rev "0.4") (company "vea.raceremote"))
 (symbol (lib_id "RaceRemote_Permit:TPS3808G33DBV") (at 76.2 88.9 0) (unit 1) (in_bom yes) (on_board yes) (dnp no) (property "Reference" "U403" (at 76.2 58.42 0) (effects (font (size 1.27 1.27))))(property "Value" "TPS3808G33DBVR" (at 76.2 55.88 0) (effects (font (size 1.27 1.27))))(property "Footprint" "" (at 76.2 88.9 0) (hide yes) (effects (font (size 1.27 1.27))))(property "Datasheet" "https://www.ti.com/lit/ds/symlink/tps3808.pdf" (at 76.2 88.9 0) (hide yes) (effects (font (size 1.27 1.27))))(pin "5")(pin "3")(pin "2")(pin "1")(pin "4")(pin "6")(instances (project "charge-permit" (path "/dee5d6a9-d751-5a9d-94e1-a01dfcba550a" (reference "U403") (unit 1)))))
 (symbol (lib_id "RaceRemote_Permit:SN74LVC2G17DCK") (at 203.2 88.9 0) (unit 1) (in_bom yes) (on_board yes) (dnp no) (property "Reference" "U402" (at 203.2 58.42 0) (effects (font (size 1.27 1.27))))(property "Value" "SN74LVC2G17DCKR" (at 203.2 55.88 0) (effects (font (size 1.27 1.27))))(property "Footprint" "" (at 203.2 88.9 0) (hide yes) (effects (font (size 1.27 1.27))))(property "Datasheet" "https://www.ti.com/lit/gpn/sn74lvc2g17" (at 203.2 88.9 0) (hide yes) (effects (font (size 1.27 1.27))))(pin "1")(pin "3")(pin "2")(pin "6")(pin "4")(pin "5")(instances (project "charge-permit" (path "/dee5d6a9-d751-5a9d-94e1-a01dfcba550a" (reference "U402") (unit 1)))))
@@
 (wire (pts (xy 76.2 199.39) (xy 76.2 207.01)) (stroke (width 0) (type default)))
 (global_label "FAULT_BUS_N" (shape passive) (at 76.2 207.01 0) (effects (font (size 1 1)) (justify left)))
-(symbol (lib_id "RaceRemote_Permit:R") (at 203.2 195.58 0) (unit 1) (in_bom yes) (on_board yes) (dnp no) (property "Reference" "R402" (at 203.2 190.5 0) (effects (font (size 1.27 1.27))))(property "Value" "10k / 1%" (at 215.9 195.58 0) (effects (font (size 1.27 1.27))))(property "Footprint" "" (at 203.2 195.58 0) (hide yes) (effects (font (size 1.27 1.27))))(property "Datasheet" "" (at 203.2 195.58 0) (hide yes) (effects (font (size 1.27 1.27))))(pin "1")(pin "2")(instances (project "charge-permit" (path "/dee5d6a9-d751-5a9d-94e1-a01dfcba550a" (reference "R402") (unit 1)))))
+(symbol (lib_id "RaceRemote_Permit:R") (at 203.2 195.58 0) (unit 1) (in_bom yes) (on_board yes) (dnp no) (property "Reference" "R402" (at 203.2 190.5 0) (effects (font (size 1.27 1.27))))(property "Value" "47k / 1%" (at 215.9 195.58 0) (effects (font (size 1.27 1.27))))(property "Footprint" "" (at 203.2 195.58 0) (hide yes) (effects (font (size 1.27 1.27))))(property "Datasheet" "" (at 203.2 195.58 0) (hide yes) (effects (font (size 1.27 1.27))))(pin "1")(pin "2")(instances (project "charge-permit" (path "/dee5d6a9-d751-5a9d-94e1-a01dfcba550a" (reference "R402") (unit 1)))))
 (wire (pts (xy 203.2 191.77) (xy 203.2 184.15)) (stroke (width 0) (type default)))
 (global_label "ARM" (shape passive) (at 203.2 184.15 0) (effects (font (size 1 1)) (justify left)))
@@
 (wire (pts (xy 558.8 119.38) (xy 558.8 124.46)) (stroke (width 0) (type default)))
 (global_label "CHG_SUPPLY_INPUT" (shape passive) (at 558.8 124.46 0) (effects (font (size 1 1)) (justify left)))
-(text "CHARGE-PERMIT-01 v0.3 - latch + regulated CD bias; complete charger NOT qualified" (at 25.4 17.78 0) (effects (font (size 2 2)) (justify left top)))
+(text "CHARGE-PERMIT-01 v0.4 - ARM pull-down 47k for MCU inverter; complete charger NOT qualified" (at 25.4 17.78 0) (effects (font (size 2 2)) (justify left top)))
 (text "FAULT_BUS_N LOW clears Q even with ARM HIGH. Releasing fault alone does not re-arm.\nD and PRE tied HIGH. Only a new ARM rising edge after reset recovery may set Q. Q-bar intentionally unused.\nExternal fault sources / MCU revoke must sink or release; never drive shared bus HIGH." (at 25.4 27.94 0) (effects (font (size 1.27 1.27)) (justify left top)))
 (text "FAULT LOW: U405 selects CHG_BIAS_3V3 directly, even when Q is unknown.\nFAULT HIGH: U405 passes U404 output. CD LOW requires Q HIGH.\nSupervisor and both muxes use CHG_BIAS_3V3; U401/U402 use AUX.\nJ401.3 is now U406 input. J404 is active-HIGH CD, NOT PERMIT_Q." (at 25.4 274.32 0) (effects (font (size 1.27 1.27)) (justify left top)))
