File: hardware/xiao-logic-power/xiao-logic-power.kicad_sch (KiCad schematic)
At the start: 15 parts, among them J1 WAVE_5V, J2 DRIVE_GND, J3 XIAO_BAT, J4 SERVICE_VBUS, J5 DRIVE_GND, U1 TPS73701DRBR, U2 LM66100DCKR

Commit message: Remove XIAO USB sense dependency with MAX40200 reverse blocking
Parts:
- removed J4: SERVICE_VBUS, symbol RaceRemote_LogicPower:Terminal
- removed R4: 10k / 1%, symbol RaceRemote_LogicPower:R
- C3, C4: value 100n / 10V X7R -> 1u / 10V X7R
- U2: value LM66100DCKR -> MAX40200AUK+T; symbol RaceRemote_LogicPower:LM66100_DCK -> RaceRemote_LogicPower:MAX40200_AUK
Connections:
- net SERVICE_VBUS is gone; now on net LDO_4V: U2.3 (EN)
- net DRIVE_GND: no longer U2.5 (ST)
- net XIAO_BAT: now also U2.5 (OUT); no longer U2.6 (VOUT)
Other:
- note added: "No J4 / USB sense wire. Native XIAO 5V/VBUS and charge-port VBUS stay separate from this circuit."
- note added: "R3 keeps LDO load above 10mA; C2>=1uF, C3/C4>=0.33uF effective. Total OUT load capacitance <=100uF."
- note added: "U2 EN tied locally to VDD. MAX40200 detects reverse bias internally; switching transient limits remain unproven."
- note added: "Use SOT23-5 limits: 175mV max drop at 500mA / 3.3V test point. WLP headline values do not apply."
- note removed: "CE compares against U2 VIN: USB present forces switch OFF. Forward body diode remains IN -> OUT."
- note removed: "J4 = native XIAO 5V/VBUS SENSE ONLY. Never join it to J1/Waveshare or the separate charge-port VBUS."
- note removed: "R3 keeps LDO load above 10mA. C2 must remain >=1uF effective. Thermal copper and all transients need validation."
- title: XIAO logic supply - DC proposal, NOT qualified -> XIAO logic supply - automatic reverse blocking proposal
