File: hardware/drive-power-carrier/drive-power-carrier.kicad_sch (KiCad schematic)
At the start: 25 parts, among them U1 TA6586 DIP8, U2 TPS73701DRBR, U3 MAX40200AUK+T

Commit message: Correct MAX40200 footprint and clearance reserve from reviewed manufacturer drawings
Parts:
- U3: footprint RaceRemote_DrivePower:SOT23_5_Provisional_U3 -> RaceRemote_DrivePower:SOT23_5_ADI_90_0174_B_U3

Commit message: Add dedicated XIAO ground landing and free traction input return
Parts:
- added H10: DRIVE_GND, RaceRemote_DrivePower:WirePad_1mm_H10, symbol RaceRemote_Motor:WirePad
Connections:
- net DRIVE_GND: now also H10.1
Other:
- note added: "H8 = qualified Waveshare +5V. H9 = XIAO BAT0 positive. H10 = XIAO ground. H5 = motor supply return. H3 = Waveshare ground."
- note removed: "H8 = qualified Waveshare +5V. H9 = XIAO BAT0 positive. H3/H5 = DRIVE_GND. No native USB VBUS wire."
